Commit message: install rplidar package, robot_localization pkg. publish /odom to the robot_localization and the urdf to the joint_state and robot_state_publisher.

File: project2/urdf/bot.urdf.xacro (robot description, xacro)
@@ -26,11 +26,11 @@
     <xacro:property name="PI" value="3.141592653589793" />
     <!-- base properties -->
-    <xacro:property name="base_width" value="0.305" />
-    <xacro:property name="base_depth" value="0.105" />
-    <xacro:property name="base_height" value="0.365" />
+    <xacro:property name="base_width" value="0.365" />
+    <xacro:property name="base_depth" value="0.305" />
+    <xacro:property name="base_height" value="0.05" />
     <xacro:property name="base_mass" value="2.0" />
     <!-- wheel properties -->
-    <xacro:property name="wheel_ygap" value="0." />
-    <xacro:property name="wheel_xoff" value="0.295" />
+    <xacro:property name="wheel_ygap" value="0.0" />
+    <xacro:property name="wheel_xoff" value="0.1" />
     <xacro:property name="wheel_radius" value="0.04" />
     <xacro:property name="wheel_width" value="0.05" />
@@ -169,5 +169,5 @@
         <parent link="base_link" />
         <child link="lidar_link" />
-        <origin xyz="0 0 ${(base_height+lidar_height)/2+lidar_zoff}" rpy="0 0 0" />
+        <origin xyz="-0.13 0 ${(base_height+lidar_height)/2+lidar_zoff}" rpy="0 0 0" />
     </joint>
     <link name="lidar_link">
